Commit message: fix samples

File: vesc_hw_interface/launch/position_test.ros2_control.xacro (robot description, xacro)
@@ -1,13 +1,23 @@
 <?xml version="1.0" encoding="UTF-8"?>
-<robot xmlns:xacro="http://www.ros.org/wiki/xacro">
+<robot xmlns:xacro="http://www.ros.org/wiki/xacro" name="test">
+  <link name="base_link"/>
+  <link name="vesc_link"/>
+  <joint name="vesc_joint" type="prismatic">
+    <parent link="base_link"/>
+    <child link="vesc_link"/>
+    <origin xyz="0 0 0" rpy="0 0 0"/>
+    <axis xyz="0 0 1"/>
+    <limit lower="-1.0" upper="1.0" velocity="10" effort="5000"/>
+  </joint>
   <ros2_control name="vesc" type="actuator">
     <hardware>
       <plugin>vesc_hw_interface/VescHwInterface</plugin>
       <param name="port">/dev/ttyACM0</param>
-      <param name="gear_ratio">0.230769</param>
+      <param name="gear_ratio">1.0</param>
       <param name="torque_const">1.0</param>
       <param name="num_hall_sensors">3</param>
+      <!--<param name="screw_lead">0.00496</param>-->
       <param name="screw_lead">1.0</param>
-      <param name="num_rotor_poles">20</param>
+      <param name="num_rotor_poles">4</param>
       <param name="servo/Kp">0.005</param>
       <param name="servo/Ki">0.005</param>
@@ -35,10 +45,10 @@
     <joint name="vesc_joint">
       <command_interface name="position">
-        <param name="min">-1</param>
-        <param name="max">1</param>
+        <param name="min">-10</param>
+        <param name="max">10</param>
       </command_interface>
       <command_interface name="velocity">
-        <param name="min">-1</param>
-        <param name="max">1</param>
+        <param name="min">-10</param>
+        <param name="max">10</param>
       </command_interface>
       <command_interface name="effort">

File: vesc_hw_interface/launch/velocity_duty_test.ros2_control.xacro (robot description, xacro)
@@ -1,8 +1,17 @@
 <?xml version="1.0" encoding="UTF-8"?>
-<robot xmlns:xacro="http://www.ros.org/wiki/xacro">
+<robot xmlns:xacro="http://www.ros.org/wiki/xacro" name="test">
+  <link name="base_link"/>
+  <link name="vesc_link"/>
+  <joint name="vesc_joint" type="continuous">
+    <parent link="base_link"/>
+    <child link="vesc_link"/>
+    <origin xyz="0 0 0" rpy="0 0 0"/>
+    <axis xyz="0 0 1"/>
+    <limit lower="-1.0" upper="1.0" velocity="10" effort="5000"/>
+  </joint>
   <ros2_control name="vesc" type="actuator">
     <hardware>
       <plugin>vesc_hw_interface/VescHwInterface</plugin>
-      <param name="port">/dev/ttyVESC_left</param>
+      <param name="port">/dev/ttyACM0</param>
       <param name="gear_ratio">0.230769</param>
       <param name="torque_const">1.0</param>
@@ -28,6 +37,6 @@
       </command_interface>
       <command_interface name="velocity">
-        <param name="min">-1</param>
-        <param name="max">1</param>
+        <param name="min">-10</param>
+        <param name="max">10</param>
       </command_interface>
       <command_interface name="effort">
